Commit message: Update xacro

File: urdf/laser_scan.xacro (robot description, xacro)
@@ -4,5 +4,5 @@
 <robot xmlns:xacro="http://www.ros.org/wiki/xacro" name="VLP-16">
   <xacro:property name="M_PI" value="3.1415926535897931" />
-  <xacro:macro name="VLP-16" params="*origin parent:=base_link name:=velodyne topic:=/scan organize_cloud:=false hz:=10 lasers:=16 samples:=920 collision_range:=0.1 min_range:=0.1 max_range:=40.0 noise:=0.001 min_angle:=-${M_PI} max_angle:=${M_PI} gpu:=false">
+  <xacro:macro name="VLP-16" params="*origin parent:=base_link name:=velodyne topic:=/scan hz:=10 samples:=920 collision_range:=0.1 min_range:=0.1 max_range:=40.0 noise:=0.001 min_angle:=-${M_PI} max_angle:=${M_PI}">
     <joint name="${name}_base_mount_joint" type="fixed">
       <xacro:insert_block name="origin" />
@@ -67,10 +67,4 @@
               <max_angle>${max_angle}</max_angle>
             </horizontal>
-            <!-- <vertical>
-              <samples>${lasers}</samples>
-              <resolution>1</resolution>
-              <min_angle>-${15.0*M_PI/180.0}</min_angle>
-              <max_angle> ${15.0*M_PI/180.0}</max_angle>
-            </vertical> -->
           </scan>
           <range>
@@ -88,8 +82,4 @@
           <topicName>${topic}</topicName>
           <frameName>${name}</frameName>
-          <!-- <organize_cloud>${organize_cloud}</organize_cloud> -->
-          <!-- <min_range>${min_range}</min_range> -->
-          <!-- <max_range>${max_range}</max_range>
-          <gaussianNoise>${noise}</gaussianNoise> -->
         </plugin>
       </sensor>
