Commit message: Update xacro

File: urdf/materials.xacro (robot description, xacro)
@@ -1,16 +1,4 @@
 <?xml version="1.0" ?>
 <robot name="xacro_properties" xmlns:xacro="http://www.ros.org/wiki/xacro" >
-  <!-- duckpod dimension -->
-  <!-- <xacro:property name="base_length" value="0.500" />
-	<xacro:property name="base_width" value="0.230" />
-	<xacro:property name="base_height" value="0.01" />
-  <xacro:property name="base_mass" value="23.26" /> -->
-  <!-- Dimension of wheel -->
-	<xacro:property name="wheel_length" value="0.02" />
-	<xacro:property name="wheel_radius" value="0.103" />
-	<xacro:property name="wheel_x" value="0.25" />
-  <xacro:property name="wheel_y" value="0.051247243897480" />
-  <xacro:property name="wheel_z" value="0.015" />
-  <xacro:property name="wheel_mass" value="2.712173066159581" />
   <!-- Constant -->
   <!-- <xacro:property name="color_silver"> -->

File: urdf/umrobot.xacro (robot description, xacro)
@@ -17,5 +17,5 @@
       <inertial>
         <origin xyz="9.858128769194324e-06 3.224621528889134e-09 0.04149809081902185" rpy="0 0 0"/>
-        <mass value="${wheel_mass}"/>
+        <mass value="7.389916078295535"/>
         <inertia ixx="0.183983" iyy="0.216397" izz="0.287255" ixy="-3e-06" iyz="-1e-06" ixz="6e-06"/>
       </inertial>
@@ -38,5 +38,5 @@
       <inertial>
         <origin xyz="-3.835820550079916e-14 -0.05124724389748092 5.204170427930421e-17" rpy="0 0 0"/>
-        <mass value="${wheel_mass}"/>
+        <mass value="2.712173066159581"/>
         <inertia ixx="0.004501" iyy="0.007469" izz="0.004501" ixy="0.0" iyz="-0.0" ixz="-0.0"/>
       </inertial>
@@ -64,5 +64,5 @@
       <inertial>
         <origin xyz="3.322342401190781e-14 0.05124724389748064 0.0" rpy="0 0 0"/>
-        <mass value="${wheel_mass}"/>
+        <mass value="2.712173066159581"/>
         <inertia ixx="0.004501" iyy="0.007469" izz="0.004501" ixy="-0.0" iyz="0.0" ixz="0.0"/>
       </inertial>
@@ -90,5 +90,5 @@
       <inertial>
         <origin xyz="-3.83026943495679e-14 -0.05124724389748081 5.551115123125783e-17" rpy="0 0 0"/>
-        <mass value="${wheel_mass}"/>
+        <mass value="2.712173066159581"/>
         <inertia ixx="0.004501" iyy="0.007469" izz="0.004501" ixy="0.0" iyz="0.0" ixz="-0.0"/>
       </inertial>

File: urdf/umrobot_gazebo.xacro (robot description, xacro)
@@ -62,6 +62,6 @@
       <rightFrontJoint>joint_RF</rightFrontJoint>
       <rightRearJoint>joint_RB</rightRearJoint>
-      <wheelSeparation>${2*wheel_y}</wheelSeparation>
-      <wheelDiameter>${2*wheel_radius}</wheelDiameter>
+      <wheelSeparation>${2*0.051247243897480}</wheelSeparation>
+      <wheelDiameter>${2*0.103}</wheelDiameter>
       <torque>20</torque>
       <commandTopic>cmd_vel</commandTopic>
@@ -80,4 +80,6 @@
       <odometryRate>50.0</odometryRate>
       <robotBaseFrame>base_footprint</robotBaseFrame>
+      <publishOdomTF>true</publishOdomTF>
+      <broadcastTF>false</broadcastTF>
     </plugin>
   </gazebo>
