Commit message: Update xacro

File: urdf/umrobot.xacro (robot description, xacro)
@@ -6,147 +6,147 @@
   ROS Package editor: Seokjun Moon -->
 <robot name="umrobot" xmlns:xacro="http://www.ros.org/wiki/xacro">
-<xacro:include filename="$(find umrobot_description)/urdf/materials.xacro" />
-<xacro:include filename="$(find umrobot_description)/urdf/umrobot_gazebo.xacro" />
-  <link name="base_footprint"/>
-  <joint name="base_joint" type="fixed">
-    <origin xyz="0 0 0" rpy="0 0 0" />
-    <parent link="base_footprint" />
-    <child link="base_link" />
-  </joint>
-  <link name="base_link">
-    <inertial>
-      <origin xyz="9.858128769194324e-06 3.224621528889134e-09 0.04149809081902185" rpy="0 0 0"/>
-      <mass value="${wheel_mass}"/>
-      <inertia ixx="0.183983" iyy="0.216397" izz="0.287255" ixy="-3e-06" iyz="-1e-06" ixz="6e-06"/>
-    </inertial>
-    <visual>
-      <origin xyz="0 0 0" rpy="0 0 0"/>
-      <geometry>
-        <mesh filename="package://umrobot_description/meshes/base_link.stl" scale="0.001 0.001 0.001"/>
-      </geometry>
-      <material name="silver"/>
-    </visual>
-    <collision>
-      <origin xyz="0 0 0" rpy="0 0 0"/>
-      <geometry>
-        <mesh filename="package://umrobot_description/meshes/base_link.stl" scale="0.001 0.001 0.001"/>
-      </geometry>
-    </collision>
-  </link>
-  <!-- Wheels -->
-  <link name="wheel_LF">
-    <inertial>
-      <origin xyz="-3.835820550079916e-14 -0.05124724389748092 5.204170427930421e-17" rpy="0 0 0"/>
-      <mass value="${wheel_mass}"/>
-      <inertia ixx="0.004501" iyy="0.007469" izz="0.004501" ixy="0.0" iyz="-0.0" ixz="-0.0"/>
-    </inertial>
-    <visual>
-      <origin xyz="0.14 0.2 0.03" rpy="0 0 0"/>
-      <geometry>
-        <mesh filename="package://umrobot_description/meshes/wheel_joint_LF.stl" scale="0.001 0.001 0.001"/>
-      </geometry>
-      <material name="silver"/>
-    </visual>
-    <collision>
-      <origin xyz="0.14 0.2 0.03" rpy="0 0 0"/>
-      <geometry>
-        <mesh filename="package://umrobot_description/meshes/wheel_joint_LF.stl" scale="0.001 0.001 0.001"/>
-      </geometry>
-    </collision>
-  </link>
-  <joint name="joint_LF" type="continuous">
-    <origin xyz="-0.14 -0.2 -0.03" rpy="0 0 0"/>
-    <parent link="base_link"/>
-    <child link="wheel_LF"/>
-    <axis xyz="0.0 1.0 0.0"/>
-  </joint>
-  <link name="wheel_RF">
-    <inertial>
-      <origin xyz="3.322342401190781e-14 0.05124724389748064 0.0" rpy="0 0 0"/>
-      <mass value="${wheel_mass}"/>
-      <inertia ixx="0.004501" iyy="0.007469" izz="0.004501" ixy="-0.0" iyz="0.0" ixz="0.0"/>
-    </inertial>
-    <visual>
-      <origin xyz="0.14 -0.2 0.03" rpy="0 0 0"/>
-      <geometry>
-        <mesh filename="package://umrobot_description/meshes/wheel_joint_RF.stl" scale="0.001 0.001 0.001"/>
-      </geometry>
-      <material name="silver"/>
-    </visual>
-    <collision>
-      <origin xyz="0.14 -0.2 0.03" rpy="0 0 0"/>
-      <geometry>
-        <mesh filename="package://umrobot_description/meshes/wheel_joint_RF.stl" scale="0.001 0.001 0.001"/>
-      </geometry>
-    </collision>
-  </link>
-  <joint name="joint_RF" type="continuous">
-    <origin xyz="-0.14 0.2 -0.03" rpy="0 0 0"/>
-    <parent link="base_link"/>
-    <child link="wheel_RF"/>
-    <axis xyz="0.0 1.0 0.0"/>
-  </joint>
-  <link name="wheel_LB">
-    <inertial>
-      <origin xyz="-3.83026943495679e-14 -0.05124724389748081 5.551115123125783e-17" rpy="0 0 0"/>
-      <mass value="${wheel_mass}"/>
-      <inertia ixx="0.004501" iyy="0.007469" izz="0.004501" ixy="0.0" iyz="0.0" ixz="-0.0"/>
-    </inertial>
-    <visual>
-      <origin xyz="-0.14 0.2 0.03" rpy="0 0 0"/>
-      <geometry>
-        <mesh filename="package://umrobot_description/meshes/wheel_joint_LB.stl" scale="0.001 0.001 0.001"/>
-      </geometry>
-      <material name="silver"/>
-    </visual>
-    <collision>
-      <origin xyz="-0.14 0.2 0.03" rpy="0 0 0"/>
-      <geometry>
-        <mesh filename="package://umrobot_description/meshes/wheel_joint_LB.stl" scale="0.001 0.001 0.001"/>
-      </geometry>
-    </collision>
-  </link>
-  <joint name="joint_LB" type="continuous">
-    <origin xyz="0.14 -0.2 -0.03" rpy="0 0 0"/>
-    <parent link="base_link"/>
-    <child link="wheel_LB"/>
-    <axis xyz="0.0 1.0 0.0"/>
-  </joint>
-  <link name="wheel_RB">
-    <inertial>
-      <origin xyz="3.322342401190781e-14 0.05124724389748081 9.367506770274758e-17" rpy="0 0 0"/>
-      <mass value="2.712173066159581"/>
-      <inertia ixx="0.004501" iyy="0.007469" izz="0.004501" ixy="-0.0" iyz="0.0" ixz="0.0"/>
-    </inertial>
-    <visual>
-      <origin xyz="-0.14 -0.2 0.03" rpy="0 0 0"/>
-      <geometry>
-        <mesh filename="package://umrobot_description/meshes/wheel_joint_RB.stl" scale="0.001 0.001 0.001"/>
-      </geometry>
-      <material name="silver"/>
-    </visual>
-    <collision>
-      <origin xyz="-0.14 -0.2 0.03" rpy="0 0 0"/>
-      <geometry>
-        <mesh filename="package://umrobot_description/meshes/wheel_joint_RB.stl" scale="0.001 0.001 0.001"/>
-      </geometry>
-    </collision>
-  </link>
-  <joint name="joint_RB" type="continuous">
-    <origin xyz="0.14 0.2 -0.03" rpy="0 0 0"/>
-    <parent link="base_link"/>
-    <child link="wheel_RB"/>
-    <axis xyz="0.0 1.0 0.0"/>
-  </joint>
-  <!-- RPLiDAR S1 Spec in VLP-16 model -->
-  <!-- <xacro:include filename="$(find velodyne_description)/urdf/VLP-16.urdf.xacro" /> -->
-  <xacro:include filename="$(find umrobot_description)/urdf/laser_scan.xacro" />
-  <VLP-16 parent="base_link" name="velodyne" topic="/scan" hz="100" samples="1875" gpu="false">
-      <origin xyz="0.0 0.0 0.1" rpy="0 0 0" />
-  </VLP-16>
-  <!-- D435 -->
-  <xacro:include filename="$(find realsense_ros_gazebo)/xacro/depthcam.xacro"/>
-  <xacro:realsense_d435 sensor_name="d435" parent_link="base_link" rate="100">
-      <origin xyz="0.225 0 0.20" rpy="0 0 0 " />
-  </xacro:realsense_d435>
+  <xacro:include filename="$(find umrobot_description)/urdf/materials.xacro" />
+  <xacro:include filename="$(find umrobot_description)/urdf/umrobot_gazebo.xacro" />
+    <link name="base_footprint"/>
+    <joint name="base_joint" type="fixed">
+      <origin xyz="0 0 0" rpy="0 0 0" />
+      <parent link="base_footprint" />
+      <child link="base_link" />
+    </joint>
+    <link name="base_link">
+      <inertial>
+        <origin xyz="9.858128769194324e-06 3.224621528889134e-09 0.04149809081902185" rpy="0 0 0"/>
+        <mass value="${wheel_mass}"/>
+        <inertia ixx="0.183983" iyy="0.216397" izz="0.287255" ixy="-3e-06" iyz="-1e-06" ixz="6e-06"/>
+      </inertial>
+      <visual>
+        <origin xyz="0 0 0" rpy="0 0 0"/>
+        <geometry>
+          <mesh filename="package://umrobot_description/meshes/base_link.stl" scale="0.001 0.001 0.001"/>
+        </geometry>
+        <material name="silver"/>
+      </visual>
+      <collision>
+        <origin xyz="0 0 0" rpy="0 0 0"/>
+        <geometry>
+          <mesh filename="package://umrobot_description/meshes/base_link.stl" scale="0.001 0.001 0.001"/>
+        </geometry>
+      </collision>
+    </link>
+    <!-- Wheels -->
+    <link name="wheel_LF">
+      <inertial>
+        <origin xyz="-3.835820550079916e-14 -0.05124724389748092 5.204170427930421e-17" rpy="0 0 0"/>
+        <mass value="${wheel_mass}"/>
+        <inertia ixx="0.004501" iyy="0.007469" izz="0.004501" ixy="0.0" iyz="-0.0" ixz="-0.0"/>
+      </inertial>
+      <visual>
+        <origin xyz="0.14 0.2 0.03" rpy="0 0 0"/>
+        <geometry>
+          <mesh filename="package://umrobot_description/meshes/wheel_joint_LF.stl" scale="0.001 0.001 0.001"/>
+        </geometry>
+        <material name="silver"/>
+      </visual>
+      <collision>
+        <origin xyz="0.14 0.2 0.03" rpy="0 0 0"/>
+        <geometry>
+          <mesh filename="package://umrobot_description/meshes/wheel_joint_LF.stl" scale="0.001 0.001 0.001"/>
+        </geometry>
+      </collision>
+    </link>
+    <joint name="joint_LF" type="continuous">
+      <origin xyz="-0.14 -0.2 -0.03" rpy="0 0 0"/>
+      <parent link="base_link"/>
+      <child link="wheel_LF"/>
+      <axis xyz="0.0 1.0 0.0"/>
+    </joint>
+    <link name="wheel_RF">
+      <inertial>
+        <origin xyz="3.322342401190781e-14 0.05124724389748064 0.0" rpy="0 0 0"/>
+        <mass value="${wheel_mass}"/>
+        <inertia ixx="0.004501" iyy="0.007469" izz="0.004501" ixy="-0.0" iyz="0.0" ixz="0.0"/>
+      </inertial>
+      <visual>
+        <origin xyz="0.14 -0.2 0.03" rpy="0 0 0"/>
+        <geometry>
+          <mesh filename="package://umrobot_description/meshes/wheel_joint_RF.stl" scale="0.001 0.001 0.001"/>
+        </geometry>
+        <material name="silver"/>
+      </visual>
+      <collision>
+        <origin xyz="0.14 -0.2 0.03" rpy="0 0 0"/>
+        <geometry>
+          <mesh filename="package://umrobot_description/meshes/wheel_joint_RF.stl" scale="0.001 0.001 0.001"/>
+        </geometry>
+      </collision>
+    </link>
+    <joint name="joint_RF" type="continuous">
+      <origin xyz="-0.14 0.2 -0.03" rpy="0 0 0"/>
+      <parent link="base_link"/>
+      <child link="wheel_RF"/>
+      <axis xyz="0.0 1.0 0.0"/>
+    </joint>
+    <link name="wheel_LB">
+      <inertial>
+        <origin xyz="-3.83026943495679e-14 -0.05124724389748081 5.551115123125783e-17" rpy="0 0 0"/>
+        <mass value="${wheel_mass}"/>
+        <inertia ixx="0.004501" iyy="0.007469" izz="0.004501" ixy="0.0" iyz="0.0" ixz="-0.0"/>
+      </inertial>
+      <visual>
+        <origin xyz="-0.14 0.2 0.03" rpy="0 0 0"/>
+        <geometry>
+          <mesh filename="package://umrobot_description/meshes/wheel_joint_LB.stl" scale="0.001 0.001 0.001"/>
+        </geometry>
+        <material name="silver"/>
+      </visual>
+      <collision>
+        <origin xyz="-0.14 0.2 0.03" rpy="0 0 0"/>
+        <geometry>
+          <mesh filename="package://umrobot_description/meshes/wheel_joint_LB.stl" scale="0.001 0.001 0.001"/>
+        </geometry>
+      </collision>
+    </link>
+    <joint name="joint_LB" type="continuous">
+      <origin xyz="0.14 -0.2 -0.03" rpy="0 0 0"/>
+      <parent link="base_link"/>
+      <child link="wheel_LB"/>
+      <axis xyz="0.0 1.0 0.0"/>
+    </joint>
+    <link name="wheel_RB">
+      <inertial>
+        <origin xyz="3.322342401190781e-14 0.05124724389748081 9.367506770274758e-17" rpy="0 0 0"/>
+        <mass value="2.712173066159581"/>
+        <inertia ixx="0.004501" iyy="0.007469" izz="0.004501" ixy="-0.0" iyz="0.0" ixz="0.0"/>
+      </inertial>
+      <visual>
+        <origin xyz="-0.14 -0.2 0.03" rpy="0 0 0"/>
+        <geometry>
+          <mesh filename="package://umrobot_description/meshes/wheel_joint_RB.stl" scale="0.001 0.001 0.001"/>
+        </geometry>
+        <material name="silver"/>
+      </visual>
+      <collision>
+        <origin xyz="-0.14 -0.2 0.03" rpy="0 0 0"/>
+        <geometry>
+          <mesh filename="package://umrobot_description/meshes/wheel_joint_RB.stl" scale="0.001 0.001 0.001"/>
+        </geometry>
+      </collision>
+    </link>
+    <joint name="joint_RB" type="continuous">
+      <origin xyz="0.14 0.2 -0.03" rpy="0 0 0"/>
+      <parent link="base_link"/>
+      <child link="wheel_RB"/>
+      <axis xyz="0.0 1.0 0.0"/>
+    </joint>
+    <!-- RPLiDAR S1 Spec in VLP-16 model -->
+    <!-- <xacro:include filename="$(find velodyne_description)/urdf/VLP-16.urdf.xacro" /> -->
+    <xacro:include filename="$(find umrobot_description)/urdf/laser_scan.xacro" />
+    <VLP-16 parent="base_link" name="velodyne" topic="/scan" hz="10" samples="920">
+        <origin xyz="0.0 0.0 0.1" rpy="0 0 0" />
+    </VLP-16>
+    <!-- D435 -->
+    <xacro:include filename="$(find realsense_ros_gazebo)/xacro/depthcam.xacro"/>
+    <xacro:realsense_d435 sensor_name="d435" parent_link="base_link" rate="100">
+        <origin xyz="0.225 0 0.20" rpy="0 0 0 " />
+    </xacro:realsense_d435>
 </robot>

Commit message: Update IMU setting

File: urdf/umrobot.xacro (robot description, xacro)
@@ -139,4 +139,11 @@
       <axis xyz="0.0 1.0 0.0"/>
     </joint>
+    <!-- IMU -->
+    <link name="imu_link"/>
+    <joint name="imu_joint" type="fixed">
+      <parent link="base_link"/>
+      <child link="imu_link"/>
+      <origin xyz="0.225 0 0.20" rpy="0 0 0"/>
+    </joint>
     <!-- RPLiDAR S1 Spec in VLP-16 model -->
     <!-- <xacro:include filename="$(find velodyne_description)/urdf/VLP-16.urdf.xacro" /> -->

File: urdf/umrobot_gazebo.xacro (robot description, xacro)
@@ -55,4 +55,13 @@
     </gazebo>
   </xacro:macro>
+  <gazebo reference="imu_link">
+    <sensor type="imu" name="imu">
+      <always_on>true</always_on>
+      <visualize>false</visualize>
+    </sensor>
+    <material>
+      <color rgba="0.5 0.5 0.5 1.0"/>
+    </material>
+  </gazebo>
   <!-- <gazebo>
     <plugin name="skid_steer_drive_controller" filename="libgazebo_ros_skid_steer_drive.so">
@@ -84,5 +93,5 @@
     </plugin>
   </gazebo>
-  <gazebo>
+  <!-- <gazebo>
     <plugin name="imu_plugin" filename="libgazebo_ros_imu.so">
       <alwaysOn>true</alwaysOn>
@@ -93,4 +102,32 @@
       <updateRate>20.0</updateRate>
     </plugin>
+  </gazebo> -->
+  <gazebo>
+    <plugin name="imu_plugin" filename="libgazebo_ros_imu.so">
+      <alwaysOn>true</alwaysOn>
+      <bodyName>imu_link</bodyName>
+      <frameName>imu_link</frameName>
+      <topicName>imu</topicName>
+      <serviceName>imu_service</serviceName>
+      <gaussianNoise>0.0</gaussianNoise>
+      <updateRate>20.0</updateRate>
+      <imu>
+        <noise>
+          <type>gaussian</type>
+          <rate>
+            <mean>0.0</mean>
+            <stddev>2e-4</stddev>
+            <bias_mean>0.0000075</bias_mean>
+            <bias_stddev>0.0000008</bias_stddev>
+          </rate>
+          <accel>
+            <mean>0.0</mean>
+            <stddev>1.7e-2</stddev>
+            <bias_mean>0.1</bias_mean>
+            <bias_stddev>0.001</bias_stddev>
+          </accel>
+        </noise>
+      </imu>
+    </plugin>
   </gazebo>
 </robot>

Commit message: Update xacro

File: urdf/umrobot.xacro (robot description, xacro)
@@ -10,7 +10,7 @@
     <link name="base_footprint"/>
     <joint name="base_joint" type="fixed">
-      <origin xyz="0 0 0" rpy="0 0 0" />
-      <parent link="base_footprint" />
-      <child link="base_link" />
+      <parent link="base_footprint"/>
+      <child link="base_link"/>
+      <origin xyz="0 0 0.01" rpy="0 0 0" />
     </joint>
     <link name="base_link">

File: urdf/umrobot_gazebo.xacro (robot description, xacro)
@@ -1,58 +1,51 @@
 <?xml version="1.0" ?>
 <robot name="umrobot" xmlns:xacro="http://www.ros.org/wiki/xacro" >
-  <!-- <xacro:property name="body_color" value="Gazebo/Silver" /> -->
-  <xacro:macro name="umrobot_sim">
-    <!-- <gazebo reference="base_link">
-      <material>${body_color}</material>
-      <mu1>0.2</mu1>
-      <mu2>0.2</mu2>
-      <selfCollide>true</selfCollide>
-      <gravity>true</gravity>
-    </gazebo> -->
-    <gazebo reference="wheel_LF">
-      <fdir1>1 0 0</fdir1>
-      <mu1>2.0</mu1>
-      <mu2>0.2</mu2>
-      <kp>1000000.0</kp>
-      <kd>100.0</kd>
-      <minDepth>0.001</minDepth>
-      <!-- <maxVel>1.0</maxVel> -->
-      <selfCollide>true</selfCollide>
-      <gravity>true</gravity>
-    </gazebo>
-    <gazebo reference="wheel_RF">
-      <fdir1>1 0 0</fdir1>
-      <mu1>2.0</mu1>
-      <mu2>0.2</mu2>
-      <kp>1000000.0</kp>
-      <kd>100.0</kd>
-      <minDepth>0.001</minDepth>
-      <!-- <maxVel>1.0</maxVel> -->
-      <selfCollide>true</selfCollide>
-      <gravity>true</gravity>
-    </gazebo>
-    <gazebo reference="wheel_LB">
-      <fdir1>1 0 0</fdir1>
-      <mu1>2.0</mu1>
-      <mu2>0.2</mu2>
-      <kp>1000000.0</kp>
-      <kd>100.0</kd>
-      <minDepth>0.001</minDepth>
-      <!-- <maxVel>1.0</maxVel> -->
-      <selfCollide>true</selfCollide>
-      <gravity>true</gravity>
-    </gazebo>
-    <gazebo reference="wheel_RB">
-      <fdir1>1 0 0</fdir1>
-      <mu1>2.0</mu1>
-      <mu2>0.2</mu2>
-      <kp>1000000.0</kp>
-      <kd>100.0</kd>
-      <minDepth>0.001</minDepth>
-      <!-- <maxVel>1.0</maxVel> -->
-      <selfCollide>true</selfCollide>
-      <gravity>true</gravity>
-    </gazebo>
-  </xacro:macro>
+  <gazebo reference="base_link">
+    <material>Gazebo/Silver</material>
+    <!-- <mu1>0.1</mu1>
+    <mu2>0.1</mu2>
+    <selfCollide>true</selfCollide>
+    <gravity>true</gravity> -->
+  </gazebo>
+  <gazebo reference="wheel_LF">
+    <mu1>0.1</mu1>
+    <mu2>0.1</mu2>
+    <kp>500000.0</kp>
+    <kd>10.0</kd>
+    <minDepth>0.001</minDepth>
+    <maxVel>0.1</maxVel>
+    <fdir1>1 0 0</fdir1>
+    <material>Gazebo/FlatBlack</material>
+  </gazebo>
+  <gazebo reference="wheel_RF">
+    <mu1>0.1</mu1>
+    <mu2>0.1</mu2>
+    <kp>500000.0</kp>
+    <kd>10.0</kd>
+    <minDepth>0.001</minDepth>
+    <maxVel>0.1</maxVel>
+    <fdir1>1 0 0</fdir1>
+    <material>Gazebo/FlatBlack</material>
+  </gazebo>
+  <gazebo reference="wheel_LB">
+    <mu1>0.1</mu1>
+    <mu2>0.1</mu2>
+    <kp>500000.0</kp>
+    <kd>10.0</kd>
+    <minDepth>0.001</minDepth>
+    <maxVel>0.1</maxVel>
+    <fdir1>1 0 0</fdir1>
+    <material>Gazebo/FlatBlack</material>
+  </gazebo>
+  <gazebo reference="wheel_RB">
+    <mu1>0.1</mu1>
+    <mu2>0.1</mu2>
+    <kp>500000.0</kp>
+    <kd>10.0</kd>
+    <minDepth>0.001</minDepth>
+    <maxVel>0.1</maxVel>
+    <fdir1>1 0 0</fdir1>
+    <material>Gazebo/FlatBlack</material>
+  </gazebo>
   <gazebo reference="imu_link">
     <sensor type="imu" name="imu">
@@ -60,7 +53,5 @@
       <visualize>false</visualize>
     </sensor>
-    <material>
-      <color rgba="0.5 0.5 0.5 1.0"/>
-    </material>
+    <material>Gazebo/Silver</material>
   </gazebo>
   <!-- <gazebo>
@@ -85,5 +76,5 @@
     <plugin name="mecanum_controller" filename="libgazebo_ros_planar_move.so">
       <commandTopic>cmd_vel</commandTopic>
-      <odometryTopic>wheel_odom</odometryTopic>
+      <odometryTopic>odom</odometryTopic>
       <odometryFrame>odom</odometryFrame>
       <odometryRate>50.0</odometryRate>
@@ -96,5 +87,5 @@
     <plugin name="imu_plugin" filename="libgazebo_ros_imu.so">
       <alwaysOn>true</alwaysOn>
-      <bodyName>base_footprint</bodyName>
+      <bodyName>imu_link</bodyName>
       <topicName>imu</topicName>
       <serviceName>imu_service</serviceName>
@@ -111,5 +102,5 @@
       <serviceName>imu_service</serviceName>
       <gaussianNoise>0.0</gaussianNoise>
-      <updateRate>20.0</updateRate>
+      <updateRate>0</updateRate>
       <imu>
         <noise>
